Commit message: m

File: src/my_robot_description/urdf/my_robot.urdf (robot description, URDF)
Before this commit: robot my_robot, 2 links, 1 joints
Links:
- added link caster_wheel, mass 0.2; collision sphere radius=0.05; visual sphere radius=0.05
- added link laser_link, mass 0.1; collision cylinder length=0.04 radius=0.05; visual cylinder length=0.04 radius=0.05
- added link right_wheel, mass 0.5; collision cylinder length=0.05 radius=0.1; visual cylinder length=0.05 radius=0.1
- link base_link: geometry collision box size=0.5 0.3 0.15; visual box size=0.5 0.3 0.15
Joints:
- added joint base_laser_joint: type fixed, parent base_link, child laser_link, origin xyz=0.2 0 0.2 rpy=0 0 0
- added joint base_right_wheel_joint: type continuous, parent base_link, child right_wheel, origin xyz=0 0.175 0.1 rpy=0 0 0, axis 0 1 0
- added joint caster_joint: type fixed, parent base_link, child caster_wheel, origin xyz=0.2 0 -0.075 rpy=0 0 0
- joint base_left_wheel_joint: origin xyz=-0.15 0.225 0 rpy=0 0 0 -> xyz=0 -0.175 0.1 rpy=0 0 0
